File: pcb/pwjsignal/pwjsignal.kicad_pcb (KiCad board)
At the start: 2 copper layers, 53.3 x 86.4 mm, 68 parts, among them J1 Strain Gauge, J10 CN10, J11 microSD_SDIO, J2 NUCLEO E5V, J3 Power In, J4 microSD, J5 CONN_LEDPWR, J6 CONN_LEDPWR, J7 CN7, J8 CN8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

Commit message: Added Rev B of board with updated filters
* This includes new Low Pass filter cutoff frequency 80kHz.
* New instrumentation amplifier for low noise
* Added test points
Parts:
- added C9: C0.1u, Capacitor_SMD:C_1206_3216Metric_Pad1.42x1.75mm_HandSolder, F.Cu at (149.8, 107.8)
- added R6: 0, Resistor_SMD:R_0603_1608Metric_Pad1.05x0.95mm_HandSolder, F.Cu at (144.1, 103.3)
- added RV2: 10, Potentiometer_SMD:Potentiometer_Bourns_3214J_Horizontal, F.Cu at (150.7, 116.7)
- C1: value C10u -> 10u
- C2: value C120u -> 120u
- C3, C4, C5, C6, C8: value C0.1u -> 0.1u
- Cb1, Cb2, Cb3, Cb4, Cb5, Cb6: value C4.7n -> 200p
- R1, R2, R3: value R120 -> 120
- R10, R11, R13, R9, Rg2: value R10K -> 10k
- R12: value R1K -> 1k
- R14, R17: value R220 -> 220
- R15, R16: value R1.6K -> 1.6k
- R19, R20: value R200K -> 200k
- R4, R5, R7, R8: value RZERO -> 0
- RV1: value R_POT10 -> 10
- Ra1, Ra2: value R47K -> 47k
- Rb1, Rb3, Rb4, Rb5, Rb6: value R1.6K -> 10k
- Rb2: value R1.6K -> 10K
- Rf1: value R6.9K -> 6.9k
- Rf2: value R5.9K -> 5.9k
- Rf3: value R29.4K -> 29.4k
- Rg1: value R100K -> 100k
- Rg3: value R20K -> 20k
- U3: value AD629ANZ -> INA118U
- moved C7 7.98 mm to (142.0, 110.7), turned to 180 degrees
- moved R1 1.44 mm to (149.9, 112.8)
- moved R2 1.44 mm to (144.6, 112.8)
- moved U3 0.97 mm to (144.1, 107.1)
- moved RV1 0.33 mm to (143.8, 116.7)
Connections:
- C7 pad 2: /+3v3 -> Net-(C7-Pad2)
- J1 pad 1: /V+ -> /V-
- J4 pad 1: /+5V -> Net-(J4-Pad1)
- J8 pad 9: /+5V -> Net-(J8-Pad9)
- R1 pad 1: /+3v3 -> Net-(R1-Pad1)
- R1 pad 2: /V- -> /V+
- R2 pad 1: /V- -> /V+
- R3 pad 1: /V+ -> /V-
- U3 pad 1: GND -> Net-(R6-Pad2)
- U3 pad 4: GND -> Net-(C7-Pad2)
Routing:
- net /+5V: track 24.6 -> 0.00 mm
- net /V-: track 9.15 -> 19.9 mm, vias 0 -> 1
- net /V+: track 19.5 -> 11.2 mm, vias 0 -> 1
- net Net-(R1-Pad1): track 0.00 -> 8.15 mm
- net /SIG_FROM_IA: track 11.9 -> 18.7 mm, vias 0 -> 1
- net Net-(R6-Pad2): track 0.00 -> 3.21 mm
- net GND: track 27.2 -> 30.2 mm, vias 21 -> 19
- net Net-(R6-Pad1): track 0.00 -> 2.87 mm
- net Net-(C7-Pad2): track 0.00 -> 2.81 mm
- net Net-(J1-Pad2): track 13.2 -> 12.1 mm
- net /+3v3: track 166.9 -> 167.6 mm
- net /ADC1_PA3: track 16.3 -> 15.7 mm, vias 0 -> 1
- net Net-(Cb3-Pad2): vias 0 -> 1
Other:
- board text added: "+5V"
- board text added: "GND"
- board text added: "PWJ Strain Logger dave@dal.ca Rev B"
- board text removed: "PWJ StrainLogger dave@dal.ca Rev. A"
